File: digiorgan.kicad_pcb (KiCad board)
At the start: 2 copper layers, 104 parts, among them J1 Barrel_Jack_Switch, J2 Conn_01_16_Male, J22 Conn_01x04_MountingPin, J23 Conn_01x08_MountingPin, J3 Conn_01x16_Male, J4 Conn_01x16_Male, J5 Conn_01_16_Male, J6 Conn_01x16_Male, J7 Conn_01x16_Male, Q1 FDN304P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

Commit message: Fix tag footprints. Add test points. Add schematic and PCB PDFs
Parts:
- added R47: 50k, Resistors_SMD:R_0805_HandSoldering, F.Cu at (226.0, 88.1)
- added R48: 50k, Resistors_SMD:R_0805_HandSoldering, F.Cu at (228.0, 88.1)
- added TP1: TestPoint, Pin_Headers:Pin_Header_Straight_1x01_Pitch1.27mm, F.Cu at (178.2, 89.0)
- added TP10: TestPoint, Pin_Headers:Pin_Header_Straight_1x01_Pitch1.27mm, F.Cu at (227.1, 54.5)
- added TP2: TestPoint, Pin_Headers:Pin_Header_Straight_1x01_Pitch1.27mm, F.Cu at (181.4, 89.0)
- added TP3: TestPoint, Pin_Headers:Pin_Header_Straight_1x01_Pitch1.27mm, F.Cu at (184.5, 89.0)
- added TP4: TestPoint, Pin_Headers:Pin_Header_Straight_1x01_Pitch1.27mm, F.Cu at (187.7, 89.0)
- added TP5: TestPoint, Pin_Headers:Pin_Header_Straight_1x01_Pitch1.27mm, F.Cu at (190.9, 89.0)
- added TP6: TestPoint, Pin_Headers:Pin_Header_Straight_1x01_Pitch1.27mm, F.Cu at (227.1, 64.3)
- added TP7: TestPoint, Pin_Headers:Pin_Header_Straight_1x01_Pitch1.27mm, F.Cu at (227.1, 61.8)
- added TP8: TestPoint, Pin_Headers:Pin_Header_Straight_1x01_Pitch1.27mm, F.Cu at (227.1, 59.4)
- added TP9: TestPoint, Pin_Headers:Pin_Header_Straight_1x01_Pitch1.27mm, F.Cu at (227.1, 57.0)
- C2, C3: footprint Capacitors_SMD:C_0805_HandSoldering -> Capacitors_Tantalum_SMD:CP_Tantalum_Case-B_EIA-3528-21_Hand
- R21, R22, R23: value R -> 1k
- moved L2 29.2 mm to (254.7, 66.2), turned to 180 degrees
- moved C18 28.8 mm to (244.6, 66.2), turned to 180 degrees
- moved C2 3.96 mm to (262.9, 70.3), turned to 270 degrees
- moved C3 3.19 mm to (260.8, 81.3), turned to 270 degrees
Connections:
- U1 pad 21: (no net) -> VBUS
- U1 pad 22: (no net) -> VPP
- U1 pad 30: (no net) -> Net-(TP6-Pad1)
- U1 pad 31: (no net) -> Net-(TP7-Pad1)
- U1 pad 32: (no net) -> Net-(TP8-Pad1)
- U1 pad 33: (no net) -> Net-(TP9-Pad1)
- U1 pad 34: (no net) -> Net-(TP10-Pad1)
- U1 pad 4: (no net) -> Net-(TP1-Pad1)
- U1 pad 5: (no net) -> Net-(TP2-Pad1)
- U1 pad 6: (no net) -> Net-(TP3-Pad1)
- U1 pad 7: (no net) -> Net-(TP4-Pad1)
- U1 pad 8: (no net) -> Net-(TP5-Pad1)
Routing:
- net VPP: track 221.7 -> 312.0 mm
- net +5V: track 223.2 -> 184.5 mm
- net Net-(TP10-Pad1): track 0.00 -> 16.3 mm
- net Net-(TP9-Pad1): track 0.00 -> 12.8 mm
- net Net-(TP8-Pad1): track 0.00 -> 9.35 mm
- net Net-(TP5-Pad1): track 0.00 -> 7.63 mm
- net +3V3: track 269.0 -> 261.4 mm, vias 6 -> 5
- net VBUS: track 90.1 -> 97.7 mm
- net Net-(TP4-Pad1): track 0.00 -> 6.90 mm
- net Net-(TP1-Pad1): track 0.00 -> 6.85 mm
- net Net-(TP7-Pad1): track 0.00 -> 6.66 mm
- net Net-(TP3-Pad1): track 0.00 -> 6.63 mm
- net Net-(TP2-Pad1): track 0.00 -> 6.58 mm
- net Net-(TP6-Pad1): track 0.00 -> 5.18 mm
- net Net-(C1-Pad1): track 11.9 -> 15.4 mm
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Other:
- board outline added: 150 x 65 mm
- board text added: "Digi Organ v1 Copyright 2021 Daniel O'Connor darius@dons.net.au"
- board text added: "Spd"
- board text removed: "Copyright 2021 Daniel O'Connor darius@dons.net.au"
- board text removed: "Speed"
